File: board.sch (KiCad schematic (older format))
At the start: 34 parts, among them J0 Battery Pads, J1 AVR-ISP-6, J2 Micro_SD_Card_Det, J3 USB_B_Micro, SW0 RESET, SW1 POWER, SW2 UP, SW3 DOWN, SW4 LEFT, SW5 RIGHT, SW6 BTN_A, SW7 BTN_B, SW8 BTN_C, U0 ATmega1284P-AU, U1 OLED, U2 MCP73831-2-OT, U3 AP7333

Commit message: Updated Layout
Parts:
- U1: footprint Pin_Headers:Pin_Header_Straight_1x07_Pitch1.27mm -> Custom Footprints:128x128_OLED
- renumbered SW2 to SW1, SW3 to SW2, SW4 to SW3, SW5 to SW4, SW6 to SW5, SW7 to SW6, SW8 to SW7, SW1 to SW8
Connections:
- net labels added: SD_CS, SD_DETECT, SD_MISO, SD_MOSI, SD_SCK
- wire segments 100 -> 110
Changed lines of the file:
@@
 F 0 "U1" H 7650 4850 60  0000 L CNN
 F 1 "OLED" H 7650 4750 60  0000 L CNN
-F 2 "Pin_Headers:Pin_Header_Straight_1x07_Pitch1.27mm" H 8000 5200 60  0001 C CNN
+F 2 "Custom Footprints:128x128_OLED" H 8000 5200 60  0001 C CNN
 F 3 "" H 8000 5200 60  0001 C CNN
 	1    8000 5200
@@
 	1    0    0    -1
 $EndComp
-Wire Wire Line
-	2050 1500 1850 1500
-Wire Wire Line
-	1850 1500 1650 1500
-Connection ~ 1850 1500
-Wire Wire Line
-	1850 1400 1850 1500
 $Comp
 L power:+3.3V #PWR0101
@@
 Text GLabel 6600 2400 2    50   Input ~ 0
 RIGHT
-Text GLabel 6600 2500 2    50   Input ~ 0
+Text GLabel 6600 2700 2    50   Input ~ 0
 BTN_A
 Text GLabel 6600 2600 2    50   Input ~ 0
 BTN_B
-Text GLabel 6600 2700 2    50   Input ~ 0
+Text GLabel 6600 2500 2    50   Input ~ 0
 BTN_C
 Wire Wire Line
@@
 Wire Wire Line
 	8200 4850 8200 5000
-Text GLabel 6600 3400 2    50   Input ~ 0
+Text GLabel 6600 3100 2    50   Input ~ 0
 D_DC
 Wire Wire Line
@@
 Wire Wire Line
 	8300 4850 8300 5000
-Text GLabel 6600 3300 2    50   Input ~ 0
+Text GLabel 6600 3000 2    50   Input ~ 0
 D_CS
 Wire Wire Line
@@
 Wire Wire Line
 	7500 5000 7700 5000
-Text GLabel 6600 3000 2    50   Input ~ 0
+Text GLabel 6600 3400 2    50   Input ~ 0
 D_SCK
 Wire Wire Line
@@
 Text GLabel 7900 4850 1    50   Input ~ 0
 D_SCK
-Text GLabel 6600 3100 2    50   Input ~ 0
+Text GLabel 6600 3300 2    50   Input ~ 0
 D_MOSI
 Wire Wire Line
@@
 Wire Wire Line
 	3750 1850 3750 1950
-Wire Wire Line
-	3250 1400 3250 1550
-Wire Wire Line
-	3250 1550 3450 1550
 $Comp
 L Custom~Library:C C2
@@
 	1    0    0    -1
 $EndComp
-Connection ~ 3250 1550
 Wire Wire Line
 	3250 1850 3250 1950
@@
 	9150 1300 8350 1300
 Connection ~ 8350 1300
-Wire Wire Line
-	8350 1600 8850 1600
-Wire Wire Line
-	8850 1600 8850 1500
-Wire Wire Line
-	8850 1500 9150 1500
-Connection ~ 8350 1600
 $Comp
 L power:GND #PWR017
@@
 $EndComp
 $Comp
-L Custom~Library:SW_DPST_x2 SW1
+L Custom~Library:SW_DPST_x2 SW8
 U 1 1 5BB38E19
 P 3250 1200
-F 0 "SW1" V 3296 1112 50  0000 R CNN
+F 0 "SW8" V 3296 1112 50  0000 R CNN
 F 1 "POWER" V 3205 1112 50  0000 R CNN
 F 2 "Buttons_Switches_SMD:SW_DIP_x1_W8.61mm_Slide_LowProfile" H 3250 1200 50  0001 C CNN
@@
 	1150 4000 1150 4700
 $Comp
-L Switch:SW_Push SW2
+L Switch:SW_Push SW1
 U 1 1 5BB3920E
 P 1350 2200
-F 0 "SW2" H 1350 2485 50  0000 C CNN
+F 0 "SW1" H 1350 2485 50  0000 C CNN
 F 1 "UP" H 1350 2394 50  0000 C CNN
 F 2 "Buttons_Switches_SMD:SW_SPST_PTS645" H 1350 2400 50  0001 C CNN
@@
 $EndComp
 $Comp
-L Switch:SW_Push SW3
+L Switch:SW_Push SW2
 U 1 1 5BB3926A
 P 1350 2800
-F 0 "SW3" H 1350 3085 50  0000 C CNN
+F 0 "SW2" H 1350 3085 50  0000 C CNN
 F 1 "DOWN" H 1350 2994 50  0000 C CNN
 F 2 "Buttons_Switches_SMD:SW_SPST_PTS645" H 1350 3000 50  0001 C CNN
@@
 	1150 2800 1150 3400
 $Comp
-L Switch:SW_Push SW4
+L Switch:SW_Push SW3
 U 1 1 5BB392C2
 P 1350 3400
-F 0 "SW4" H 1350 3685 50  0000 C CNN
+F 0 "SW3" H 1350 3685 50  0000 C CNN
 F 1 "LEFT" H 1350 3594 50  0000 C CNN
 F 2 "Buttons_Switches_SMD:SW_SPST_PTS645" H 1350 3600 50  0001 C CNN
@@
 	1150 3400 1150 4000
 $Comp
-L Switch:SW_Push SW5
+L Switch:SW_Push SW4
 U 1 1 5BB39320
 P 1350 4000
-F 0 "SW5" H 1350 4285 50  0000 C CNN
+F 0 "SW4" H 1350 4285 50  0000 C CNN
 F 1 "RIGHT" H 1350 4194 50  0000 C CNN
 F 2 "Buttons_Switches_SMD:SW_SPST_PTS645" H 1350 4200 50  0001 C CNN
@@
 $EndComp
 $Comp
-L Switch:SW_Push SW6
+L Switch:SW_Push SW5
 U 1 1 5BB3937A
 P 1350 4700
-F 0 "SW6" H 1350 4985 50  0000 C CNN
+F 0 "SW5" H 1350 4985 50  0000 C CNN
 F 1 "BTN_A" H 1350 4894 50  0000 C CNN
 F 2 "Buttons_Switches_SMD:SW_SPST_PTS645" H 1350 4900 50  0001 C CNN
@@
 	1150 4700 1150 5300
 $Comp
-L Switch:SW_Push SW7
+L Switch:SW_Push SW6
 U 1 1 5BB393E2
 P 1350 5300
-F 0 "SW7" H 1350 5585 50  0000 C CNN
+F 0 "SW6" H 1350 5585 50  0000 C CNN
 F 1 "BTN_B" H 1350 5494 50  0000 C CNN
 F 2 "Buttons_Switches_SMD:SW_SPST_PTS645" H 1350 5500 50  0001 C CNN
@@
 	1150 5300 1150 5900
 $Comp
-L Switch:SW_Push SW8
+L Switch:SW_Push SW7
 U 1 1 5BB39448
 P 1350 5900
-F 0 "SW8" H 1350 6185 50  0000 C CNN
+F 0 "SW7" H 1350 6185 50  0000 C CNN
 F 1 "BTN_C" H 1350 6094 50  0000 C CNN
 F 2 "Buttons_Switches_SMD:SW_SPST_PTS645" H 1350 6100 50  0001 C CNN
@@
 Wire Wire Line
 	2550 2300 2550 2450
+Text GLabel 9150 1600 0    50   Input ~ 0
+SD_MISO
+Text GLabel 9150 1200 0    50   Input ~ 0
+SD_MOSI
+Wire Wire Line
+	8350 1600 8650 1600
+Wire Wire Line
+	8650 1600 8650 1500
+Wire Wire Line
+	8650 1500 9150 1500
+Connection ~ 8350 1600
+Text GLabel 9150 1400 0    50   Input ~ 0
+SD_SCK
+Text GLabel 9150 1100 0    50   Input ~ 0
+SD_CS
+Text GLabel 9150 1800 0    50   Input ~ 0
+SD_DETECT
+$Comp
+L power:+3.3V #PWR0103
+U 1 1 5BAE7783
+P 8900 2150
+F 0 "#PWR0103" H 8900 2000 50  0001 C CNN
+F 1 "+3.3V" H 8915 2323 50  0000 C CNN
+F 2 "" H 8900 2150 50  0001 C CNN
+F 3 "" H 8900 2150 50  0001 C CNN
+	1    8900 2150
+	1    0    0    -1
+$EndComp
+Wire Wire Line
+	9150 1900 9150 2150
+Wire Wire Line
+	9150 2150 8900 2150
+$Comp
+L power:GND #PWR0104
+U 1 1 5BAED575
+P 8650 1000
+F 0 "#PWR0104" H 8650 750 50  0001 C CNN
+F 1 "GND" H 8655 827 50  0000 C CNN
+F 2 "" H 8650 1000 50  0001 C CNN
+F 3 "" H 8650 1000 50  0001 C CNN
+	1    8650 1000
+	1    0    0    -1
+$EndComp
+Wire Wire Line
+	8650 1000 9150 1000
+Wire Wire Line
+	9150 1700 8650 1700
+Wire Wire Line
+	8650 1700 8650 1600
+Connection ~ 8650 1600
+Text GLabel 6600 4200 2    50   Input ~ 0
+SD_CS
+Text GLabel 6600 3900 2    50   Input ~ 0
+SD_SCK
+Text GLabel 6600 4000 2    50   Input ~ 0
+SD_MOSI
+Text GLabel 6600 4100 2    50   Input ~ 0
+SD_MISO
+Text GLabel 6600 4300 2    50   Input ~ 0
+SD_DETECT
+Wire Wire Line
+	6450 3900 6600 3900
+Wire Wire Line
+	6450 4000 6600 4000
+Wire Wire Line
+	6450 4100 6600 4100
+Wire Wire Line
+	6450 4200 6600 4200
+Wire Wire Line
+	6450 4300 6600 4300
+Wire Wire Line
+	2050 1500 1850 1500
+Wire Wire Line
+	1850 1400 1850 1500
+Connection ~ 1850 1500
+Wire Wire Line
+	1850 1500 1650 1500
+Wire Wire Line
+	3250 1400 3250 1550
+Wire Wire Line
+	3450 1550 3250 1550
+Connection ~ 3250 1550
 $EndSCHEMATC

Commit message: Added tracks
Parts:
- added R9: 1K, Resistors_SMD:R_0805, symbol Custom~Library:R
Connections:
- wire segments 110 -> 113
Changed lines of the file:
@@
 Text GLabel 9150 1100 0    50   Input ~ 0
 SD_CS
-Text GLabel 9150 1800 0    50   Input ~ 0
+Text GLabel 8500 1950 0    50   Input ~ 0
 SD_DETECT
 $Comp
@@
 Text GLabel 6600 4200 2    50   Input ~ 0
 SD_CS
+Text GLabel 6600 4000 2    50   Input ~ 0
+SD_SCK
+Text GLabel 6600 4100 2    50   Input ~ 0
+SD_MOSI
 Text GLabel 6600 3900 2    50   Input ~ 0
-SD_SCK
-Text GLabel 6600 4000 2    50   Input ~ 0
-SD_MOSI
-Text GLabel 6600 4100 2    50   Input ~ 0
 SD_MISO
 Text GLabel 6600 4300 2    50   Input ~ 0
@@
 	3450 1550 3250 1550
 Connection ~ 3250 1550
+Wire Wire Line
+	8500 1950 8650 1950
+Wire Wire Line
+	8650 1950 8650 1800
+Wire Wire Line
+	8650 1800 9150 1800
+$Comp
+L Custom~Library:R R9
+U 1 1 5BB3D25D
+P 8650 2100
+F 0 "R9" H 8720 2146 50  0000 L CNN
+F 1 "1K" H 8720 2055 50  0000 L CNN
+F 2 "Resistors_SMD:R_0805" V 8580 2100 50  0001 C CNN
+F 3 "" H 8650 2100 50  0001 C CNN
+	1    8650 2100
+	1    0    0    -1
+$EndComp
+Connection ~ 8650 1950
+$Comp
+L power:GND #PWR0105
+U 1 1 5BB3D2ED
+P 8650 2250
+F 0 "#PWR0105" H 8650 2000 50  0001 C CNN
+F 1 "GND" H 8655 2077 50  0000 C CNN
+F 2 "" H 8650 2250 50  0001 C CNN
+F 3 "" H 8650 2250 50  0001 C CNN
+	1    8650 2250
+	1    0    0    -1
+$EndComp
 $EndSCHEMATC

Commit message: added crystal
Parts:
- added C7, C8: 22pF, Capacitors_SMD:C_0805, symbol Device:C
- added Y1: 16MHz, Crystals:Crystal_SMD_7050-4pin_7.0x5.0mm, symbol Device:Crystal_Small
- J1: value AVR-ISP-6 -> PGRM
- J2: value Micro_SD_Card_Det -> Micro SD Slot
- U0: value ATmega1284P-AU -> ATmega1284P
- U2: value MCP73831-2-OT -> CHG
- U3: value AP7333 -> Reg
Connections:
- wire segments 113 -> 122
Changed lines of the file:
@@
 P 5850 3800
 F 0 "U0" H 5350 5750 50  0000 L BNN
-F 1 "ATmega1284P-AU" H 5950 1850 50  0000 L TNN
+F 1 "ATmega1284P" H 5950 1850 50  0000 L TNN
 F 2 "Housings_QFP:TQFP-44_10x10mm_Pitch0.8mm" H 5850 3800 50  0001 C CIN
 F 3 "http://ww1.microchip.com/downloads/en/DeviceDoc/Atmel-8272-8-bit-AVR-microcontroller-ATmega164A_PA-324A_PA-644A_PA-1284_P_datasheet.pdf" H 5850 3800 50  0001 C CNN
@@
 P 10050 3200
 F 0 "J1" V 9850 3450 50  0000 C CNN
-F 1 "AVR-ISP-6" V 9700 3250 50  0000 C CNN
+F 1 "PGRM" V 9700 3250 50  0000 C CNN
 F 2 "Pin_Headers:Pin_Header_Straight_2x03_Pitch1.27mm" V 9800 3250 50  0001 C CNN
 F 3 " ~" H 8775 2650 50  0001 C CNN
@@
 P 10050 1400
 F 0 "J2" H 10000 2217 50  0000 C CNN
-F 1 "Micro_SD_Card_Det" H 10000 2126 50  0000 C CNN
+F 1 "Micro SD Slot" H 10000 2126 50  0000 C CNN
 F 2 "Connectors_Card:Hirose_DM3AT-SF-PEJM5" H 12100 2100 50  0001 C CNN
 F 3 "https://www.hirose.com/product/en/download_file/key_name/DM3/category/Catalog/doc_file_id/49662/?file_category_id=4&item_id=195&is_series=1" H 10050 1500 50  0001 C CNN
@@
 P 3750 1550
 F 0 "U3" H 3750 1792 50  0000 C CNN
-F 1 "AP7333" H 3750 1701 50  0000 C CNN
+F 1 "Reg" H 3750 1701 50  0000 C CNN
 F 2 "TO_SOT_Packages_SMD:SOT-23" H 3750 1775 50  0001 C CIN
 F 3 "http://www.tme.eu/fr/Document/ced3461ed31ea70a3c416fb648e0cde7/APE8865-3.pdf" H 3750 1550 50  0001 C CNN
@@
 P 3500 3450
 F 0 "U2" H 3500 3928 50  0000 C CNN
-F 1 "MCP73831-2-OT" H 3500 3837 50  0000 C CNN
+F 1 "CHG" H 3500 3837 50  0000 C CNN
 F 2 "TO_SOT_Packages_SMD:SOT-23-5" H 3550 3200 50  0001 L CIN
 F 3 "http://ww1.microchip.com/downloads/en/DeviceDoc/20001984g.pdf" H 3350 3400 50  0001 C CNN
@@
 	1    0    0    -1
 $EndComp
+$Comp
+L Device:Crystal_Small Y1
+U 1 1 5BBCEB00
+P 5000 2400
+F 0 "Y1" V 4954 2312 50  0000 R CNN
+F 1 "16MHz" V 5045 2312 50  0000 R CNN
+F 2 "Crystals:Crystal_SMD_7050-4pin_7.0x5.0mm" H 5000 2400 50  0001 C CNN
+F 3 "~" H 5000 2400 50  0001 C CNN
+	1    5000 2400
+	0    -1   1    0
+$EndComp
+Wire Wire Line
+	5000 2300 5250 2300
+Wire Wire Line
+	5000 2500 5250 2500
+$Comp
+L Device:C C7
+U 1 1 5BBD9858
+P 4600 2250
+F 0 "C7" V 4348 2250 50  0000 C CNN
+F 1 "22pF" V 4439 2250 50  0000 C CNN
+F 2 "Capacitors_SMD:C_0805" H 4638 2100 50  0001 C CNN
+F 3 "~" H 4600 2250 50  0001 C CNN
+	1    4600 2250
+	0    1    1    0
+$EndComp
+$Comp
+L Device:C C8
+U 1 1 5BBD9934
+P 4600 2550
+F 0 "C8" V 4348 2550 50  0000 C CNN
+F 1 "22pF" V 4439 2550 50  0000 C CNN
+F 2 "Capacitors_SMD:C_0805" H 4638 2400 50  0001 C CNN
+F 3 "~" H 4600 2550 50  0001 C CNN
+	1    4600 2550
+	0    1    1    0
+$EndComp
+Wire Wire Line
+	4750 2250 5000 2250
+Wire Wire Line
+	5000 2250 5000 2300
+Connection ~ 5000 2300
+Wire Wire Line
+	4750 2550 5000 2550
+Wire Wire Line
+	5000 2550 5000 2500
+Connection ~ 5000 2500
+$Comp
+L power:GND #PWR03
+U 1 1 5BBE1528
+P 4200 2400
+F 0 "#PWR03" H 4200 2150 50  0001 C CNN
+F 1 "GND" H 4205 2227 50  0000 C CNN
+F 2 "" H 4200 2400 50  0001 C CNN
+F 3 "" H 4200 2400 50  0001 C CNN
+	1    4200 2400
+	1    0    0    -1
+$EndComp
+Wire Wire Line
+	4200 2400 4450 2400
+Wire Wire Line
+	4450 2400 4450 2250
+Wire Wire Line
+	4450 2550 4450 2400
+Connection ~ 4450 2400
 $EndSCHEMATC

Commit message: Revert "added crystal"
This reverts commit 60f505991b0e3ccfce5c63fb45a6584053ac2d9c.
Parts:
- removed C7, C8: 22pF, Capacitors_SMD:C_0805, symbol Device:C
- removed Y1: 16MHz, Crystals:Crystal_SMD_7050-4pin_7.0x5.0mm, symbol Device:Crystal_Small
- J1: value PGRM -> AVR-ISP-6
- J2: value Micro SD Slot -> Micro_SD_Card_Det
- U0: value ATmega1284P -> ATmega1284P-AU
- U2: value CHG -> MCP73831-2-OT
- U3: value Reg -> AP7333
Connections:
- wire segments 122 -> 113
Changed lines of the file:
@@
 P 5850 3800
 F 0 "U0" H 5350 5750 50  0000 L BNN
-F 1 "ATmega1284P" H 5950 1850 50  0000 L TNN
+F 1 "ATmega1284P-AU" H 5950 1850 50  0000 L TNN
 F 2 "Housings_QFP:TQFP-44_10x10mm_Pitch0.8mm" H 5850 3800 50  0001 C CIN
 F 3 "http://ww1.microchip.com/downloads/en/DeviceDoc/Atmel-8272-8-bit-AVR-microcontroller-ATmega164A_PA-324A_PA-644A_PA-1284_P_datasheet.pdf" H 5850 3800 50  0001 C CNN
@@
 P 10050 3200
 F 0 "J1" V 9850 3450 50  0000 C CNN
-F 1 "PGRM" V 9700 3250 50  0000 C CNN
+F 1 "AVR-ISP-6" V 9700 3250 50  0000 C CNN
 F 2 "Pin_Headers:Pin_Header_Straight_2x03_Pitch1.27mm" V 9800 3250 50  0001 C CNN
 F 3 " ~" H 8775 2650 50  0001 C CNN
@@
 P 10050 1400
 F 0 "J2" H 10000 2217 50  0000 C CNN
-F 1 "Micro SD Slot" H 10000 2126 50  0000 C CNN
+F 1 "Micro_SD_Card_Det" H 10000 2126 50  0000 C CNN
 F 2 "Connectors_Card:Hirose_DM3AT-SF-PEJM5" H 12100 2100 50  0001 C CNN
 F 3 "https://www.hirose.com/product/en/download_file/key_name/DM3/category/Catalog/doc_file_id/49662/?file_category_id=4&item_id=195&is_series=1" H 10050 1500 50  0001 C CNN
@@
 P 3750 1550
 F 0 "U3" H 3750 1792 50  0000 C CNN
-F 1 "Reg" H 3750 1701 50  0000 C CNN
+F 1 "AP7333" H 3750 1701 50  0000 C CNN
 F 2 "TO_SOT_Packages_SMD:SOT-23" H 3750 1775 50  0001 C CIN
 F 3 "http://www.tme.eu/fr/Document/ced3461ed31ea70a3c416fb648e0cde7/APE8865-3.pdf" H 3750 1550 50  0001 C CNN
@@
 P 3500 3450
 F 0 "U2" H 3500 3928 50  0000 C CNN
-F 1 "CHG" H 3500 3837 50  0000 C CNN
+F 1 "MCP73831-2-OT" H 3500 3837 50  0000 C CNN
 F 2 "TO_SOT_Packages_SMD:SOT-23-5" H 3550 3200 50  0001 L CIN
 F 3 "http://ww1.microchip.com/downloads/en/DeviceDoc/20001984g.pdf" H 3350 3400 50  0001 C CNN
@@
 	1    0    0    -1
 $EndComp
-$Comp
-L Device:Crystal_Small Y1
-U 1 1 5BBCEB00
-P 5000 2400
-F 0 "Y1" V 4954 2312 50  0000 R CNN
-F 1 "16MHz" V 5045 2312 50  0000 R CNN
-F 2 "Crystals:Crystal_SMD_7050-4pin_7.0x5.0mm" H 5000 2400 50  0001 C CNN
-F 3 "~" H 5000 2400 50  0001 C CNN
-	1    5000 2400
-	0    -1   1    0
-$EndComp
-Wire Wire Line
-	5000 2300 5250 2300
-Wire Wire Line
-	5000 2500 5250 2500
-$Comp
-L Device:C C7
-U 1 1 5BBD9858
-P 4600 2250
-F 0 "C7" V 4348 2250 50  0000 C CNN
-F 1 "22pF" V 4439 2250 50  0000 C CNN
-F 2 "Capacitors_SMD:C_0805" H 4638 2100 50  0001 C CNN
-F 3 "~" H 4600 2250 50  0001 C CNN
-	1    4600 2250
-	0    1    1    0
-$EndComp
-$Comp
-L Device:C C8
-U 1 1 5BBD9934
-P 4600 2550
-F 0 "C8" V 4348 2550 50  0000 C CNN
-F 1 "22pF" V 4439 2550 50  0000 C CNN
-F 2 "Capacitors_SMD:C_0805" H 4638 2400 50  0001 C CNN
-F 3 "~" H 4600 2550 50  0001 C CNN
-	1    4600 2550
-	0    1    1    0
-$EndComp
-Wire Wire Line
-	4750 2250 5000 2250
-Wire Wire Line
-	5000 2250 5000 2300
-Connection ~ 5000 2300
-Wire Wire Line
-	4750 2550 5000 2550
-Wire Wire Line
-	5000 2550 5000 2500
-Connection ~ 5000 2500
-$Comp
-L power:GND #PWR03
-U 1 1 5BBE1528
-P 4200 2400
-F 0 "#PWR03" H 4200 2150 50  0001 C CNN
-F 1 "GND" H 4205 2227 50  0000 C CNN
-F 2 "" H 4200 2400 50  0001 C CNN
-F 3 "" H 4200 2400 50  0001 C CNN
-	1    4200 2400
-	1    0    0    -1
-$EndComp
-Wire Wire Line
-	4200 2400 4450 2400
-Wire Wire Line
-	4450 2400 4450 2250
-Wire Wire Line
-	4450 2550 4450 2400
-Connection ~ 4450 2400
 $EndSCHEMATC

Commit message: Changed labels
Parts:
- J1: value AVR-ISP-6 -> PGRM
- J2: value Micro_SD_Card_Det -> Micro SD Slot
- U0: value ATmega1284P-AU -> ATmega1284P
- U2: value MCP73831-2-OT -> CHG
- U3: value AP7333 -> Reg
Changed lines of the file:
@@
 P 5850 3800
 F 0 "U0" H 5350 5750 50  0000 L BNN
-F 1 "ATmega1284P-AU" H 5950 1850 50  0000 L TNN
+F 1 "ATmega1284P" H 5950 1850 50  0000 L TNN
 F 2 "Housings_QFP:TQFP-44_10x10mm_Pitch0.8mm" H 5850 3800 50  0001 C CIN
 F 3 "http://ww1.microchip.com/downloads/en/DeviceDoc/Atmel-8272-8-bit-AVR-microcontroller-ATmega164A_PA-324A_PA-644A_PA-1284_P_datasheet.pdf" H 5850 3800 50  0001 C CNN
@@
 P 10050 3200
 F 0 "J1" V 9850 3450 50  0000 C CNN
-F 1 "AVR-ISP-6" V 9700 3250 50  0000 C CNN
+F 1 "PGRM" V 9700 3250 50  0000 C CNN
 F 2 "Pin_Headers:Pin_Header_Straight_2x03_Pitch1.27mm" V 9800 3250 50  0001 C CNN
 F 3 " ~" H 8775 2650 50  0001 C CNN
@@
 P 10050 1400
 F 0 "J2" H 10000 2217 50  0000 C CNN
-F 1 "Micro_SD_Card_Det" H 10000 2126 50  0000 C CNN
+F 1 "Micro SD Slot" H 10000 2126 50  0000 C CNN
 F 2 "Connectors_Card:Hirose_DM3AT-SF-PEJM5" H 12100 2100 50  0001 C CNN
 F 3 "https://www.hirose.com/product/en/download_file/key_name/DM3/category/Catalog/doc_file_id/49662/?file_category_id=4&item_id=195&is_series=1" H 10050 1500 50  0001 C CNN
@@
 P 3750 1550
 F 0 "U3" H 3750 1792 50  0000 C CNN
-F 1 "AP7333" H 3750 1701 50  0000 C CNN
+F 1 "Reg" H 3750 1701 50  0000 C CNN
 F 2 "TO_SOT_Packages_SMD:SOT-23" H 3750 1775 50  0001 C CIN
 F 3 "http://www.tme.eu/fr/Document/ced3461ed31ea70a3c416fb648e0cde7/APE8865-3.pdf" H 3750 1550 50  0001 C CNN
@@
 P 3500 3450
 F 0 "U2" H 3500 3928 50  0000 C CNN
-F 1 "MCP73831-2-OT" H 3500 3837 50  0000 C CNN
+F 1 "CHG" H 3500 3837 50  0000 C CNN
 F 2 "TO_SOT_Packages_SMD:SOT-23-5" H 3550 3200 50  0001 L CIN
 F 3 "http://ww1.microchip.com/downloads/en/DeviceDoc/20001984g.pdf" H 3350 3400 50  0001 C CNN

Commit message: Revert "Revert "added crystal""
This reverts commit 7f3a5123c106fe465dc47a4e88f841c035e49e56.
Parts:
- added C7, C8: 22pF, Capacitors_SMD:C_0805, symbol Device:C
- added Y1: 16MHz, Crystals:Crystal_SMD_7050-4pin_7.0x5.0mm, symbol Device:Crystal_Small
Connections:
- wire segments 113 -> 122
Changed lines of the file:
@@
 	1    0    0    -1
 $EndComp
+$Comp
+L Device:Crystal_Small Y1
+U 1 1 5BBCEB00
+P 5000 2400
+F 0 "Y1" V 4954 2312 50  0000 R CNN
+F 1 "16MHz" V 5045 2312 50  0000 R CNN
+F 2 "Crystals:Crystal_SMD_7050-4pin_7.0x5.0mm" H 5000 2400 50  0001 C CNN
+F 3 "~" H 5000 2400 50  0001 C CNN
+	1    5000 2400
+	0    -1   1    0
+$EndComp
+Wire Wire Line
+	5000 2300 5250 2300
+Wire Wire Line
+	5000 2500 5250 2500
+$Comp
+L Device:C C7
+U 1 1 5BBD9858
+P 4600 2250
+F 0 "C7" V 4348 2250 50  0000 C CNN
+F 1 "22pF" V 4439 2250 50  0000 C CNN
+F 2 "Capacitors_SMD:C_0805" H 4638 2100 50  0001 C CNN
+F 3 "~" H 4600 2250 50  0001 C CNN
+	1    4600 2250
+	0    1    1    0
+$EndComp
+$Comp
+L Device:C C8
+U 1 1 5BBD9934
+P 4600 2550
+F 0 "C8" V 4348 2550 50  0000 C CNN
+F 1 "22pF" V 4439 2550 50  0000 C CNN
+F 2 "Capacitors_SMD:C_0805" H 4638 2400 50  0001 C CNN
+F 3 "~" H 4600 2550 50  0001 C CNN
+	1    4600 2550
+	0    1    1    0
+$EndComp
+Wire Wire Line
+	4750 2250 5000 2250
+Wire Wire Line
+	5000 2250 5000 2300
+Connection ~ 5000 2300
+Wire Wire Line
+	4750 2550 5000 2550
+Wire Wire Line
+	5000 2550 5000 2500
+Connection ~ 5000 2500
+$Comp
+L power:GND #PWR03
+U 1 1 5BBE1528
+P 4200 2400
+F 0 "#PWR03" H 4200 2150 50  0001 C CNN
+F 1 "GND" H 4205 2227 50  0000 C CNN
+F 2 "" H 4200 2400 50  0001 C CNN
+F 3 "" H 4200 2400 50  0001 C CNN
+	1    4200 2400
+	1    0    0    -1
+$EndComp
+Wire Wire Line
+	4200 2400 4450 2400
+Wire Wire Line
+	4450 2400 4450 2250
+Wire Wire Line
+	4450 2550 4450 2400
+Connection ~ 4450 2400
 $EndSCHEMATC

Commit message: sorted crystal
I think. Got into a proper pickle there.
Parts:
- Y1: footprint Crystals:Crystal_SMD_7050-4pin_7.0x5.0mm -> Crystals:Crystal_SMD_5032-2pin_5.0x3.2mm
Changed lines of the file:
@@
 F 0 "Y1" V 4954 2312 50  0000 R CNN
 F 1 "16MHz" V 5045 2312 50  0000 R CNN
-F 2 "Crystals:Crystal_SMD_7050-4pin_7.0x5.0mm" H 5000 2400 50  0001 C CNN
+F 2 "Crystals:Crystal_SMD_5032-2pin_5.0x3.2mm" H 5000 2400 50  0001 C CNN
 F 3 "~" H 5000 2400 50  0001 C CNN
 	1    5000 2400

Commit message: reworked to be MCU agnostic
Parts:
- removed C0, C4: 1uF, Capacitors_SMD:C_0805, symbol Custom~Library:C
- removed C7, C8: 22pF, Capacitors_SMD:C_0805, symbol Device:C
- removed J1: PGRM, Pin_Headers:Pin_Header_Straight_2x03_Pitch1.27mm, symbol Connector:AVR-ISP-6
- removed J2: Micro SD Slot, Connectors_Card:Hirose_DM3AT-SF-PEJM5, symbol Connector:Micro_SD_Card_Det
- removed R9: 1K, Resistors_SMD:R_0805, symbol Custom~Library:R
- removed U0: ATmega1284P, Housings_QFP:TQFP-44_10x10mm_Pitch0.8mm, symbol MCU_Microchip_ATmega:ATmega1284P-AU
- removed Y1: 16MHz, Crystals:Crystal_SMD_5032-2pin_5.0x3.2mm, symbol Device:Crystal_Small
- added C4: 1uF, Capacitor_THT:C_Rect_L7.0mm_W2.5mm_P5.00mm, symbol Device:C
- added J1: Shard, Connector_PinHeader_2.54mm:PinHeader_2x10_P2.54mm_Vertical, symbol Connector_Generic:Conn_02x10_Odd_Even
- added R9: 10k, Resistor_THT:R_Axial_DIN0207_L6.3mm_D2.5mm_P7.62mm_Horizontal, symbol Device:R
- C1, C2, C3, C5, C6: footprint Capacitors_SMD:C_0805 -> Capacitor_THT:C_Rect_L7.0mm_W2.5mm_P5.00mm; symbol Custom~Library:C -> Device:C
- J2: renamed from J3; value USB_B_Micro -> USB-Micro; footprint Connectors_USB:USB_Micro-B_Molex-105017-0001 -> Connector_USB:USB_Micro-B_Molex-105017-0001
- R0, R1, R2, R3, R4, R5, R6, R7, R8: footprint Resistors_SMD:R_0805 -> Resistor_THT:R_Axial_DIN0207_L6.3mm_D2.5mm_P7.62mm_Horizontal; symbol Custom~Library:R -> Device:R
- SW0, SW1, SW2, SW3, SW4, SW5, SW6, SW7: footprint Buttons_Switches_SMD:SW_SPST_PTS645 -> Button_Switch_THT:SW_PUSH_6mm
- SW8: footprint Buttons_Switches_SMD:SW_DIP_x1_W8.61mm_Slide_LowProfile -> Button_Switch_THT:SW_DIP_SPSTx01_Slide_9.78x4.72mm_W7.62mm_P2.54mm; symbol Custom~Library:SW_DPST_x2 -> Switch:SW_SPST
- U1: footprint Custom Footprints:128x128_OLED -> Custom Footprints:128x128-OLED
- U2: footprint TO_SOT_Packages_SMD:SOT-23-5 -> Package_TO_SOT_SMD:SOT-23-5
- U3: footprint TO_SOT_Packages_SMD:SOT-23 -> Package_TO_SOT_SMD:SOT-23
Connections:
- net labels added: D+, D-
- net labels removed: MISO, MOSI, SCK, SD_CS, SD_DETECT, SD_MISO, SD_MOSI, SD_SCK
- wire segments 122 -> 93
Other:
- moved on the sheet: J0
