File: board.kicad_pcb (KiCad board)
At the start: 2 copper layers, 85.3 x 35.3 mm, 32 parts, among them J0 Battery, J1 Shard, J2 USB-Micro, SW0 RESET, SW1 UP, SW2 DOWN, SW3 LEFT, SW4 RIGHT, SW5 BTN_A, SW6 BTN_B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

Commit message: flipped logo to match shard
Parts:
- moved SPIKE 16.6 mm to (150.5, 86.3), turned to 225 degrees
Changed lines of the file:
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@@
   )
   (module SPIKE (layer B.Cu)
-    (at 162.25 98 135)
-    (fp_text reference SPIKE (at 3.5 -1.5 135) (layer B.Fab) hide
+    (at 150.5 86.3 225)
+    (fp_text reference SPIKE (at 3.5 -1.5 225) (layer B.Fab) hide
       (effects (font (size 1.524 1.524) (thickness 0.3)) (justify mirror))
     )
-    (fp_text value "" (at 0 0 135) (layer B.SilkS)
+    (fp_text value "" (at 0 0 225) (layer B.SilkS)
       (effects (font (size 1.27 1.27) (thickness 0.15)) (justify mirror))
     )
